File: i5ether2.0/SPI_module.kicad_sch (KiCad schematic)
At the start: 0 parts

Commit message: Pcb huellas y esquematico (sin resitensias)
Parts:
- added J3: Conn_02x03_Counter_Clockwise, Connector_IDC:IDC-Header_2x04_P2.54mm_Vertical, symbol Connector_Generic:Conn_02x03_Counter_Clockwise
Connections:
- new net CSn: J3.3 (Pin_3)
- new net GND: J3.1 (Pin_1)
- new net RX: J3.2 (Pin_2)
- new net SCK: J3.4 (Pin_4)
- new net TX: J3.5 (Pin_5)
- no-connect marks 0 -> 1
Changed lines of the file:
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@@
 (kicad_sch (version 20230121) (generator eeschema)
   (paper "A4")
+  (no_connect (at 147.32 93.98))
+  (wire (pts (xy 129.54 96.52) (xy 134.62 96.52))
+    (stroke (width 0) (type default))
+  )
+  (wire (pts (xy 147.32 96.52) (xy 151.13 96.52))
+    (stroke (width 0) (type default))
+  )
+  (wire (pts (xy 129.54 93.98) (xy 134.62 93.98))
+    (stroke (width 0) (type default))
+  )
+  (wire (pts (xy 147.32 99.06) (xy 151.13 99.06))
+    (stroke (width 0) (type default))
+  )
+  (wire (pts (xy 129.54 99.06) (xy 134.62 99.06))
+    (stroke (width 0) (type default))
+  )
+  (hierarchical_label "CSn" (shape input) (at 129.54 99.06 180) (fields_autoplaced)
+    (effects (font (size 1.27 1.27)) (justify right))
+  )
+  (hierarchical_label "TX" (shape input) (at 151.13 96.52 0) (fields_autoplaced)
+    (effects (font (size 1.27 1.27)) (justify left))
+  )
+  (hierarchical_label "RX" (shape input) (at 129.54 96.52 180) (fields_autoplaced)
+    (effects (font (size 1.27 1.27)) (justify right))
+  )
+  (hierarchical_label "SCK" (shape input) (at 151.13 99.06 0) (fields_autoplaced)
+    (effects (font (size 1.27 1.27)) (justify left))
+  )
+  (symbol (lib_id "Connector_Generic:Conn_02x03_Counter_Clockwise") (at 139.7 96.52 0) (unit 1)
+    (in_bom yes) (on_board yes) (dnp no) (fields_autoplaced)
+    (property "Reference" "J3" (at 140.97 88.9 0)
+      (effects (font (size 1.27 1.27)))
+    )
+    (property "Value" "Conn_02x03_Counter_Clockwise" (at 140.97 91.44 0)
+      (effects (font (size 1.27 1.27)))
+    )
+    (property "Footprint" "Connector_IDC:IDC-Header_2x04_P2.54mm_Vertical" (at 139.7 96.52 0)
+      (effects (font (size 1.27 1.27)) hide)
+    )
+    (property "Datasheet" "~" (at 139.7 96.52 0)
+      (effects (font (size 1.27 1.27)) hide)
+    )
+    (pin "1")
+    (pin "2")
+    (pin "3")
+    (pin "4")
+    (pin "5")
+    (pin "6")
+    (instances
+      (project "i5ether"
+        (path "/8004154c-2cb0-4a38-a510-aadf61b39ef8/2eb1c9aa-8378-460a-af5f-78d29c0155ac"
+          (reference "J3") (unit 1)
+        )
+      )
+    )
+  )
+  (symbol (lib_id "power:GND") (at 129.54 93.98 270) (unit 1)
+    (in_bom yes) (on_board yes) (dnp no) (fields_autoplaced)
+    (property "Reference" "#PWR03" (at 123.19 93.98 0)
+      (effects (font (size 1.27 1.27)) hide)
+    )
+    (property "Value" "GND" (at 125.73 94.615 90)
+      (effects (font (size 1.27 1.27)) (justify right))
+    )
+    (property "Footprint" "" (at 129.54 93.98 0)
+      (effects (font (size 1.27 1.27)) hide)
+    )
+    (property "Datasheet" "" (at 129.54 93.98 0)
+      (effects (font (size 1.27 1.27)) hide)
+    )
+    (pin "1")
+    (instances
+      (project "i5ether"
+        (path "/8004154c-2cb0-4a38-a510-aadf61b39ef8/2eb1c9aa-8378-460a-af5f-78d29c0155ac"
+          (reference "#PWR03") (unit 1)
+        )
+      )
+    )
+  )
 )
