File: i5ether2.0/bluetooth_module.kicad_sch (KiCad schematic)
At the start: 0 parts

Commit message: Pcb huellas y esquematico (sin resitensias)
Parts:
- added J4: Conn_01x04, Connector_PinHeader_2.54mm:PinHeader_1x04_P2.54mm_Horizontal, symbol Connector_Generic:Conn_01x04
Connections:
- new net +3.3V: J4.4 (Pin_4)
- new net GND: J4.3 (Pin_3)
- new net RX: J4.1 (Pin_1)
- new net TX: J4.2 (Pin_2)
Changed lines of the file:
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@@
 (kicad_sch (version 20230121) (generator eeschema)
   (paper "A4")
+  (wire (pts (xy 134.62 101.6) (xy 142.24 101.6))
+    (stroke (width 0) (type default))
+  )
+  (wire (pts (xy 134.62 99.06) (xy 142.24 99.06))
+    (stroke (width 0) (type default))
+  )
+  (wire (pts (xy 133.35 104.14) (xy 142.24 104.14))
+    (stroke (width 0) (type default))
+  )
+  (wire (pts (xy 134.62 96.52) (xy 142.24 96.52))
+    (stroke (width 0) (type default))
+  )
+  (hierarchical_label "TX" (shape input) (at 134.62 99.06 180) (fields_autoplaced)
+    (effects (font (size 1.27 1.27)) (justify right))
+  )
+  (hierarchical_label "RX" (shape input) (at 134.62 96.52 180) (fields_autoplaced)
+    (effects (font (size 1.27 1.27)) (justify right))
+  )
+  (symbol (lib_id "Connector_Generic:Conn_01x04") (at 147.32 99.06 0) (unit 1)
+    (in_bom yes) (on_board yes) (dnp no) (fields_autoplaced)
+    (property "Reference" "J4" (at 149.86 99.695 0)
+      (effects (font (size 1.27 1.27)) (justify left))
+    )
+    (property "Value" "Conn_01x04" (at 149.86 102.235 0)
+      (effects (font (size 1.27 1.27)) (justify left))
+    )
+    (property "Footprint" "Connector_PinHeader_2.54mm:PinHeader_1x04_P2.54mm_Horizontal" (at 147.32 99.06 0)
+      (effects (font (size 1.27 1.27)) hide)
+    )
+    (property "Datasheet" "~" (at 147.32 99.06 0)
+      (effects (font (size 1.27 1.27)) hide)
+    )
+    (pin "1")
+    (pin "2")
+    (pin "3")
+    (pin "4")
+    (instances
+      (project "i5ether"
+        (path "/8004154c-2cb0-4a38-a510-aadf61b39ef8/0943df1d-0e2b-40e0-83c6-b1dbbad7a2f6"
+          (reference "J4") (unit 1)
+        )
+      )
+    )
+  )
+  (symbol (lib_id "power:GND") (at 134.62 101.6 270) (unit 1)
+    (in_bom yes) (on_board yes) (dnp no) (fields_autoplaced)
+    (property "Reference" "#PWR04" (at 128.27 101.6 0)
+      (effects (font (size 1.27 1.27)) hide)
+    )
+    (property "Value" "GND" (at 130.81 102.235 90)
+      (effects (font (size 1.27 1.27)) (justify right))
+    )
+    (property "Footprint" "" (at 134.62 101.6 0)
+      (effects (font (size 1.27 1.27)) hide)
+    )
+    (property "Datasheet" "" (at 134.62 101.6 0)
+      (effects (font (size 1.27 1.27)) hide)
+    )
+    (pin "1")
+    (instances
+      (project "i5ether"
+        (path "/8004154c-2cb0-4a38-a510-aadf61b39ef8/0943df1d-0e2b-40e0-83c6-b1dbbad7a2f6"
+          (reference "#PWR04") (unit 1)
+        )
+      )
+    )
+  )
+  (symbol (lib_id "power:+3.3V") (at 133.35 104.14 90) (unit 1)
+    (in_bom yes) (on_board yes) (dnp no) (fields_autoplaced)
+    (property "Reference" "#PWR05" (at 137.16 104.14 0)
+      (effects (font (size 1.27 1.27)) hide)
+    )
+    (property "Value" "+3.3V" (at 129.54 104.775 90)
+      (effects (font (size 1.27 1.27)) (justify left))
+    )
+    (property "Footprint" "" (at 133.35 104.14 0)
+      (effects (font (size 1.27 1.27)) hide)
+    )
+    (property "Datasheet" "" (at 133.35 104.14 0)
+      (effects (font (size 1.27 1.27)) hide)
+    )
+    (pin "1")
+    (instances
+      (project "i5ether"
+        (path "/8004154c-2cb0-4a38-a510-aadf61b39ef8/0943df1d-0e2b-40e0-83c6-b1dbbad7a2f6"
+          (reference "#PWR05") (unit 1)
+        )
+      )
+    )
+  )
 )
