File: i5ether2.0/screen_module.kicad_sch (KiCad schematic)
At the start: 1 part, among them J1 Conn_01x14

Commit message: Avances en placa
Parts:
- J1: footprint (none) -> Connector_PinHeader_2.54mm:PinHeader_1x14_P2.54mm_Vertical
Changed lines of the file:
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@@
       (effects (font (size 1.27 1.27)) (justify left) hide)
     )
-    (property "Footprint" "" (at 143.51 91.44 0)
+    (property "Footprint" "Connector_PinHeader_2.54mm:PinHeader_1x14_P2.54mm_Vertical" (at 143.51 91.44 0)
       (effects (font (size 1.27 1.27)) hide)
     )

Commit message: Pcb huellas y esquematico (sin resitensias)
Parts:
- J1: footprint Connector_PinHeader_2.54mm:PinHeader_1x14_P2.54mm_Vertical -> Connector_IDC:IDC-Header_2x08-1MP_P2.54mm_Latch6.5mm_Vertical
Changed lines of the file:
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@@
       (effects (font (size 1.27 1.27)) (justify left) hide)
     )
-    (property "Footprint" "Connector_PinHeader_2.54mm:PinHeader_1x14_P2.54mm_Vertical" (at 143.51 91.44 0)
+    (property "Footprint" "Connector_IDC:IDC-Header_2x08-1MP_P2.54mm_Latch6.5mm_Vertical" (at 143.51 91.44 0)
       (effects (font (size 1.27 1.27)) hide)
     )
