File: i5ether3.0/bluetooth_module.kicad_sch (KiCad schematic)
At the start: 1 part, among them J4 Conn_01x04

Commit message: PCB corecciones
Parts:
- J4: footprint Connector_PinHeader_2.54mm:PinHeader_1x04_P2.54mm_Horizontal -> Connector_PinSocket_2.54mm:PinSocket_1x04_P2.54mm_Horizontal
Connections:
- net +3.3V: now also J4.1 (Pin_1); no longer J4.4 (Pin_4)
- net GND: now also J4.2 (Pin_2); no longer J4.3 (Pin_3)
- net RX: now also J4.4 (Pin_4); no longer J4.1 (Pin_1)
- net TX: now also J4.3 (Pin_3); no longer J4.2 (Pin_2)
Changed lines of the file:
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@@
 (kicad_sch (version 20230121) (generator eeschema)
   (paper "A4")
-  (wire (pts (xy 134.62 101.6) (xy 142.24 101.6))
+  (wire (pts (xy 135.89 96.52) (xy 142.24 96.52))
     (stroke (width 0) (type default))
   )
-  (wire (pts (xy 134.62 99.06) (xy 142.24 99.06))
+  (wire (pts (xy 135.89 99.06) (xy 142.24 99.06))
     (stroke (width 0) (type default))
   )
-  (wire (pts (xy 133.35 104.14) (xy 142.24 104.14))
+  (wire (pts (xy 135.89 101.6) (xy 142.24 101.6))
     (stroke (width 0) (type default))
   )
-  (wire (pts (xy 134.62 96.52) (xy 142.24 96.52))
+  (wire (pts (xy 135.89 104.14) (xy 142.24 104.14))
     (stroke (width 0) (type default))
   )
-  (hierarchical_label "TX" (shape input) (at 134.62 99.06 180) (fields_autoplaced)
+  (hierarchical_label "TX" (shape input) (at 135.89 101.6 180) (fields_autoplaced)
     (effects (font (size 1.27 1.27)) (justify right))
   )
-  (hierarchical_label "RX" (shape input) (at 134.62 96.52 180) (fields_autoplaced)
+  (hierarchical_label "RX" (shape input) (at 135.89 104.14 180) (fields_autoplaced)
     (effects (font (size 1.27 1.27)) (justify right))
   )
@@
       (effects (font (size 1.27 1.27)) (justify left))
     )
-    (property "Footprint" "Connector_PinHeader_2.54mm:PinHeader_1x04_P2.54mm_Horizontal" (at 147.32 99.06 0)
+    (property "Footprint" "Connector_PinSocket_2.54mm:PinSocket_1x04_P2.54mm_Horizontal" (at 147.32 99.06 0)
       (effects (font (size 1.27 1.27)) hide)
     )
@@
     )
   )
-  (symbol (lib_id "power:GND") (at 134.62 101.6 270) (unit 1)
+  (symbol (lib_id "power:GND") (at 135.89 99.06 270) (unit 1)
     (in_bom yes) (on_board yes) (dnp no) (fields_autoplaced)
-    (property "Reference" "#PWR04" (at 128.27 101.6 0)
+    (property "Reference" "#PWR04" (at 129.54 99.06 0)
       (effects (font (size 1.27 1.27)) hide)
     )
-    (property "Value" "GND" (at 130.81 102.235 90)
+    (property "Value" "GND" (at 132.08 99.695 90)
       (effects (font (size 1.27 1.27)) (justify right))
     )
-    (property "Footprint" "" (at 134.62 101.6 0)
+    (property "Footprint" "" (at 135.89 99.06 0)
       (effects (font (size 1.27 1.27)) hide)
     )
-    (property "Datasheet" "" (at 134.62 101.6 0)
+    (property "Datasheet" "" (at 135.89 99.06 0)
       (effects (font (size 1.27 1.27)) hide)
     )
@@
     )
   )
-  (symbol (lib_id "power:+3.3V") (at 133.35 104.14 90) (unit 1)
+  (symbol (lib_id "power:+3.3V") (at 135.89 96.52 90) (unit 1)
     (in_bom yes) (on_board yes) (dnp no) (fields_autoplaced)
-    (property "Reference" "#PWR05" (at 137.16 104.14 0)
+    (property "Reference" "#PWR05" (at 139.7 96.52 0)
       (effects (font (size 1.27 1.27)) hide)
     )
-    (property "Value" "+3.3V" (at 129.54 104.775 90)
+    (property "Value" "+3.3V" (at 132.08 97.155 90)
       (effects (font (size 1.27 1.27)) (justify left))
     )
-    (property "Footprint" "" (at 133.35 104.14 0)
+    (property "Footprint" "" (at 135.89 96.52 0)
       (effects (font (size 1.27 1.27)) hide)
     )
-    (property "Datasheet" "" (at 133.35 104.14 0)
+    (property "Datasheet" "" (at 135.89 96.52 0)
       (effects (font (size 1.27 1.27)) hide)
     )
