File: i5ether3.0/i5ether.kicad_sch (KiCad schematic)
At the start: 5 parts, among them P1 Conn_02x15_Counter_Clockwise, P2 Conn_02x15_Counter_Clockwise, P3 Conn_02x15_Counter_Clockwise, P4 Conn_02x15_Counter_Clockwise, P6 Conn_02x15_Counter_Clockwise

Commit message: PCB corecciones
Parts:
- removed P6: Conn_02x15_Counter_Clockwise, Connector_PinHeader_2.54mm:PinHeader_2x15_P2.54mm_Vertical, symbol Connector_Generic:Conn_02x15_Counter_Clockwise
- added P5: Conn_02x15_Counter_Clockwise, Connector_PinHeader_2.54mm:PinHeader_2x15_P2.54mm_Vertical, symbol Connector_Generic:Conn_02x15_Counter_Clockwise
Connections:
- net screen_module/GND is gone; now on net screen_module/T_CS: P2.4 (Pin_4)
- net screen_module/LED is gone; now on net screen_module/CS: P2.7 (Pin_7)
- net screen_module/T_CLK is gone; now on net +3.3V: P2.11 (Pin_11)
- net screen_module/T_DO is gone; now on net GND: P2.28 (Pin_28)
- net screen_module/VCC is gone; now on net screen_module/SDO(MISO): P2.2 (Pin_2)
- net SPI_module/CSn: now also P4.22 (Pin_22); no longer P4.12 (Pin_12)
- net SPI_module/RX: now also P4.24 (Pin_24); no longer P4.10 (Pin_10)
- net SPI_module/SCK: now also P4.26 (Pin_26); no longer P4.8 (Pin_8)
- net SPI_module/TX: now also P4.20 (Pin_20); no longer P4.6 (Pin_6)
- net bluetooth_module/RX: now also P4.6 (Pin_6)
- net bluetooth_module/TX: now also P4.4 (Pin_4)
- net ethernet_module/GLED-: now also P5.2 (Pin_2); no longer P2.23 (Pin_23)
- net ethernet_module/RD+: now also P1.26 (Pin_26); no longer P1.23 (Pin_23)
- net ethernet_module/RD-: now also P1.24 (Pin_24); no longer P1.25 (Pin_25)
- net ethernet_module/TD+: now also P1.20 (Pin_20); no longer P1.19 (Pin_19)
- net ethernet_module/TD-: now also P1.22 (Pin_22); no longer P1.21 (Pin_21)
- net ethernet_module/YLED-: now also P5.1 (Pin_1); no longer P2.25 (Pin_25)
- net screen_module/CS: no longer P2.6 (Pin_6)
- net screen_module/DC: now also P2.6 (Pin_6); no longer P2.10 (Pin_10)
- net screen_module/SDI(MOSI): now also P2.3 (Pin_3); no longer P2.12 (Pin_12)
- net screen_module/SDO(MISO): no longer P2.9 (Pin_9)
- net screen_module/T_CS: no longer P2.24 (Pin_24)
- net screen_module/T_IRQ: now also P2.1 (Pin_1); no longer P2.30 (Pin_30)
- net GND: now reaches P2.15 (Pin_15)
- net GND: now also P1.10 (Pin_10), P1.15 (Pin_15), P1.27 (Pin_27), P1.28 (Pin_28), P1.9 (Pin_9), P2.10 (Pin_10), P2.27 (Pin_27), P2.9 (Pin_9), P3.10 (Pin_10), P3.15 (Pin_15), P3.27 (Pin_27), P3.28 (Pin_28), P3.9 (Pin_9), P4.10 (Pin_10), P4.15 (Pin_15), P4.27 (Pin_27), P4.28 (Pin_28), P4.9 (Pin_9), P5.10 (Pin_10), P5.15 (Pin_15), P5.27 (Pin_27), P5.28 (Pin_28), P5.9 (Pin_9)
- net +5V: now reaches P2.16 (Pin_16)
- net +5V: now also P1.16 (Pin_16), P3.16 (Pin_16), P4.16 (Pin_16), P5.16 (Pin_16)
- net +3.3V: now reaches P2.29 (Pin_29)
- net +3.3V: now also P1.11 (Pin_11), P1.12 (Pin_12), P1.29 (Pin_29), P1.30 (Pin_30), P2.12 (Pin_12), P2.30 (Pin_30), P3.11 (Pin_11), P3.12 (Pin_12), P3.29 (Pin_29), P3.30 (Pin_30), P4.11 (Pin_11), P4.12 (Pin_12), P4.29 (Pin_29), P4.30 (Pin_30), P5.11 (Pin_11), P5.12 (Pin_12), P5.29 (Pin_29), P5.30 (Pin_30)
- net screen_module/RESET: no longer names the net of P2.8 (Pin_8)
- net screen_module/T_DIN: no longer names the net of P2.26 (Pin_26)
- no-connect marks 124 -> 81
Other:
- sheet screen_module ports: added none; removed GND, VCC
- moved on the sheet: P1, P2, P4
