File: i5ether3.0/screen_module.kicad_sch (KiCad schematic)
At the start: 1 part, among them J1 Conn_01x14

Commit message: PCB corecciones
Connections:
- net VCC renamed +3.3V
Changed lines of the file:
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@@
-    (effects (font (size 1.27 1.27)) (justify right))
-  )
-  (hierarchical_label "VCC" (shape input) (at 132.08 109.22 180) (fields_autoplaced)
     (effects (font (size 1.27 1.27)) (justify right))
   )
@@
   )
   (hierarchical_label "SCK" (shape input) (at 132.08 93.98 180) (fields_autoplaced)
-    (effects (font (size 1.27 1.27)) (justify right))
-  )
-  (hierarchical_label "GND" (shape input) (at 132.08 106.68 180) (fields_autoplaced)
     (effects (font (size 1.27 1.27)) (justify right))
   )
@@
         )
       )
+    )
+  )
+  (symbol (lib_id "power:+3.3V") (at 132.08 109.22 90) (unit 1)
+    (in_bom yes) (on_board yes) (dnp no) (fields_autoplaced)
+    (property "Reference" "#PWR032" (at 135.89 109.22 0)
+      (effects (font (size 1.27 1.27)) hide)
+    )
+    (property "Value" "+3.3V" (at 128.27 109.855 90)
+      (effects (font (size 1.27 1.27)) (justify left))
+    )
+    (property "Footprint" "" (at 132.08 109.22 0)
+      (effects (font (size 1.27 1.27)) hide)
+    )
+    (property "Datasheet" "" (at 132.08 109.22 0)
+      (effects (font (size 1.27 1.27)) hide)
+    )
+    (pin "1")
+    (instances
+      (project "i5ether"
+        (path "/8004154c-2cb0-4a38-a510-aadf61b39ef8/3146e5f8-bf0e-4709-b480-36018c22d70a"
+          (reference "#PWR032") (unit 1)
+        )
+      )
+    )
+  )
+  (symbol (lib_id "power:GND") (at 132.08 106.68 270) (unit 1)
+    (in_bom yes) (on_board yes) (dnp no) (fields_autoplaced)
+    (property "Reference" "#PWR031" (at 125.73 106.68 0)
+      (effects (font (size 1.27 1.27)) hide)
+    )
+    (property "Value" "GND" (at 128.27 107.315 90)
+      (effects (font (size 1.27 1.27)) (justify right))
+    )
+    (property "Footprint" "" (at 132.08 106.68 0)
+      (effects (font (size 1.27 1.27)) hide)
+    )
+    (property "Datasheet" "" (at 132.08 106.68 0)
+      (effects (font (size 1.27 1.27)) hide)
+    )
+    (pin "1")
+    (instances
+      (project "i5ether"
+        (path "/8004154c-2cb0-4a38-a510-aadf61b39ef8/3146e5f8-bf0e-4709-b480-36018c22d70a"
+          (reference "#PWR031") (unit 1)
+        )
+      )
