File: PCB/i5ether.kicad_pcb (KiCad board)
At the start: 2 copper layers, 100 x 75 mm, 15 parts, among them J1 Conn_01x14, J2 7499011121A, J3 Conn_02x03_Counter_Clockwise, J4 Conn_01x04, P1 Conn_02x15_Counter_Clockwise, P2 Conn_02x15_Counter_Clockwise, P3 Conn_02x15_Counter_Clockwise, P4 Conn_02x15_Counter_Clockwise, P5 Conn_02x15_Counter_Clockwise

Commit message: PCB_Final
Parts:
- added G***: LOGO, Logo:UNCargador_Logo, F.Cu at (147.9, 114.6)
